File: board/board.kicad_pcb (KiCad board)
At the start: 2 copper layers, 21 x 13 mm, 1 part

Commit message: initial
Parts:
- added C1: 56nF, Capacitor_SMD:C_0402_1005Metric, F.Cu at (147.5, 108.3)
- added C10: 22pF, Capacitor_SMD:C_0402_1005Metric, F.Cu at (153.9, 109.5)
- added C11: 100nF, Capacitor_SMD:C_0603_1608Metric, F.Cu at (153.9, 103.5)
- added C12: 56nF, Capacitor_SMD:C_0402_1005Metric, F.Cu at (154.4, 108.0)
- added C13: 56nF, Capacitor_SMD:C_0402_1005Metric, F.Cu at (158.0, 105.5)
- added C14: 100nF, Capacitor_SMD:C_0603_1608Metric, F.Cu at (158.5, 110.0)
- added C15: 22pF, Capacitor_SMD:C_0402_1005Metric, F.Cu at (158.5, 104.0)
- added C16: 56nF, Capacitor_SMD:C_0402_1005Metric, F.Cu at (159.0, 105.5)
- added C2: 22pF, Capacitor_SMD:C_0402_1005Metric, F.Cu at (147.0, 109.7)
- added C3: 100nF, Capacitor_SMD:C_0603_1608Metric, F.Cu at (147.0, 103.5)
- added C4: 56nF, Capacitor_SMD:C_0402_1005Metric, F.Cu at (146.5, 108.3)
- added C5: 56nF, Capacitor_SMD:C_0402_1005Metric, F.Cu at (151.3, 105.4)
- added C6: 100nF, Capacitor_SMD:C_0603_1608Metric, F.Cu at (150.8, 110.1)
- added C7: 22pF, Capacitor_SMD:C_0402_1005Metric, F.Cu at (150.8, 103.8)
- added C8: 56nF, Capacitor_SMD:C_0402_1005Metric, F.Cu at (150.3, 105.4)
- added C9: 56nF, Capacitor_SMD:C_0402_1005Metric, F.Cu at (153.4, 108.0)
- added J1: 009_Ethernet_Cable_side, on_edge:on_edge_2x05_device, F.Cu at (140.0, 112.5)
- added J2: 009_Ethernet_Cable_side, on_edge:on_edge_2x05_device, F.Cu at (140.0, 96.5)
- added R1: 49.9R, Resistor_SMD:R_0402_1005Metric, F.Cu at (147.5, 106.3)
- added R10: 49.9R, Resistor_SMD:R_0402_1005Metric, F.Cu at (158.0, 107.5)
- added R11: 100R, Resistor_SMD:R_0402_1005Metric, F.Cu at (158.5, 103.0)
- added R12: 49.9R, Resistor_SMD:R_0402_1005Metric, F.Cu at (159.0, 107.5)
- added R2: 100R, Resistor_SMD:R_0402_1005Metric, F.Cu at (147.0, 110.7)
- added R3: 49.9R, Resistor_SMD:R_0402_1005Metric, F.Cu at (146.5, 106.3)
- added R4: 49.9R, Resistor_SMD:R_0402_1005Metric, F.Cu at (151.3, 107.3)
- added R5: 100R, Resistor_SMD:R_0402_1005Metric, F.Cu at (150.8, 102.8)
- added R6: 49.9R, Resistor_SMD:R_0402_1005Metric, F.Cu at (150.3, 107.3)
- added R7: 49.9R, Resistor_SMD:R_0402_1005Metric, F.Cu at (153.4, 106.0)
- added R8: 100R, Resistor_SMD:R_0402_1005Metric, F.Cu at (153.9, 110.5)
- added R9: 49.9R, Resistor_SMD:R_0402_1005Metric, F.Cu at (154.4, 106.0)
- moved LOGO1 7.75 mm to (156.2, 94.3)
Routing:
- net /implementation/GND: track 0.00 -> 52.2 mm, vias 0 -> 7
- net /implementation/RXN3: track 0.00 -> 27.3 mm, vias 0 -> 1
- net /implementation/RXP3: track 0.00 -> 23.9 mm, vias 0 -> 1
- net /implementation/RXP2: track 0.00 -> 23.5 mm, vias 0 -> 1
- net /implementation/RXN2: track 0.00 -> 23.2 mm, vias 0 -> 1
- net /implementation/TXN3: track 0.00 -> 21.4 mm, vias 0 -> 1
- net /implementation/TXP3: track 0.00 -> 21.4 mm, vias 0 -> 1
- net /implementation/RXP0: track 0.00 -> 17.0 mm, vias 0 -> 2
- net /implementation/RXN1: track 0.00 -> 17.0 mm
- net /implementation/RXN0: track 0.00 -> 16.3 mm, vias 0 -> 2
- net /implementation/TXP2: track 0.00 -> 16.1 mm, vias 0 -> 1
- net /implementation/RXP1: track 0.00 -> 15.2 mm
- net /implementation/TXN2: track 0.00 -> 14.1 mm, vias 0 -> 1
- net /implementation/TXP1: track 0.00 -> 13.3 mm, vias 0 -> 2
- net /implementation/TXN1: track 0.00 -> 13.3 mm
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Other:
- board size 21 x 13 mm -> 21 x 29 mm
