File: board/board.kicad_pcb (KiCad board)
At the start: 2 copper layers, 21 x 29 mm, 31 parts, among them J1 009_Ethernet_Cable_side, J2 009_Ethernet_Cable_side

Commit message: initial
Parts:
- moved LOGO1 2.12 mm to (156.5, 96.5)
Connections:
- net /implementation/GND renamed GND
- net /implementation/RXN0 renamed /phy2phy/RXN0
- net /implementation/RXN1 renamed /phy2phy/RXN1
- net /implementation/RXN2 renamed /phy2phy/RXN2
- net /implementation/RXN3 renamed /phy2phy/RXN3
- net /implementation/RXP0 renamed /phy2phy/RXP0
- net /implementation/RXP1 renamed /phy2phy/RXP1
- net /implementation/RXP2 renamed /phy2phy/RXP2
- net /implementation/RXP3 renamed /phy2phy/RXP3
- net /implementation/TXN0 renamed /phy2phy/TXN0
- net /implementation/TXN1 renamed /phy2phy/TXN1
- net /implementation/TXN2 renamed /phy2phy/TXN2
- net /implementation/TXN3 renamed /phy2phy/TXN3
- net /implementation/TXP0 renamed /phy2phy/TXP0
- net /implementation/TXP1 renamed /phy2phy/TXP1
- net /implementation/TXP2 renamed /phy2phy/TXP2
- net /implementation/TXP3 renamed /phy2phy/TXP3
Routing:
- net GND: vias 7 -> 45
- added copper zone on B.Cu, net GND
- added copper zone on F.Cu, net GND
Other:
- board text added: "osf.009"
- board text added: "osf.b127.v1.0"

Commit message: added JLC production data
Parts:
- C1, C12, C13, C16, C4, C5, C8, C9: value 56nF -> 100nF
- C11, C14, C3, C6: footprint Capacitor_SMD:C_0603_1608Metric -> Capacitor_SMD:C_0402_1005Metric
