File: board/board.kicad_sch (KiCad schematic)
At the start: 3 parts, among them J1 009_Ethernet_Cable_side, J2 009_Ethernet_Cable_side

Commit message: initial
Connections:
- net phy2phy/GND renamed GND
Changed lines of the file:
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@@
     (pin "9")
+  )
+  (symbol (lib_id "power:GND") (at 174.625 133.985 0) (unit 1)
+    (in_bom yes) (on_board yes) (fields_autoplaced)
+    (property "Reference" "#PWR?" (id 0) (at 174.625 140.335 0)
+      (effects (font (size 1.27 1.27)) hide)
+    )
+    (property "Value" "GND" (id 1) (at 174.625 138.43 0))
+    (property "Footprint" "" (id 2) (at 174.625 133.985 0)
+      (effects (font (size 1.27 1.27)) hide)
+    )
+    (property "Datasheet" "" (id 3) (at 174.625 133.985 0)
+      (effects (font (size 1.27 1.27)) hide)
+    )
+    (pin "1")
   )
   (symbol (lib_id "Graphic:Logo_Open_Hardware_Small") (at 273.05 157.48 0) (unit 1)
@@
   )
   (symbol_instances
+    (path "/b3361342-4700-4dca-91d7-56a7fb286888"
+      (reference "#PWR?") (unit 1) (value "GND") (footprint "")
+    )
     (path "/767ce4c6-0e55-4543-92f0-34cb8237a544/0768ff9b-bfec-4d10-8d35-adc6f13cd19a"
       (reference "C1") (unit 1) (value "56nF") (footprint "Capacitor_SMD:C_0402_1005Metric")
