File: board/phy2phy.kicad_sch (KiCad schematic)
At the start: 28 parts

Commit message: initial
Parts:
- C1, C12, C13, C16, C4, C5, C8, C9: value (none) -> 56nF; footprint (none) -> Capacitor_SMD:C_0402_1005Metric
- C10, C15, C2, C7: value (none) -> 22pF; footprint (none) -> Capacitor_SMD:C_0402_1005Metric
- C11, C14, C3, C6: value (none) -> 100nF; footprint (none) -> Capacitor_SMD:C_0603_1608Metric
- R1, R10, R12, R3, R4, R6, R7, R9: value (none) -> 49.9R; footprint (none) -> Resistor_SMD:R_0402_1005Metric
- R11, R2, R5, R8: value (none) -> 100R; footprint (none) -> Resistor_SMD:R_0402_1005Metric

Commit message: added JLC production data
Parts:
- C1, C12, C13, C16, C4, C5, C8, C9: value 56nF -> 100nF; lcsc (none) -> C307331
- C10, C15, C2, C7: lcsc (none) -> C1555
- C11, C14, C3, C6: footprint Capacitor_SMD:C_0603_1608Metric -> Capacitor_SMD:C_0402_1005Metric; lcsc (none) -> C307331
- R1, R10, R12, R3, R4, R6, R7, R9: lcsc (none) -> C25120
- R11, R2, R5, R8: lcsc (none) -> C25076
